Commit message: Code copied from constructsim. Does not run

File: catkin_ws/src/KUKA_150/kr150_description/urdf/kr150_2.xacro (robot description, xacro)
@@ -1,4 +1,4 @@
 <?xml version="1.0"?>
-<robot name="kuka_kr150_robot" xmlns:xacro="http://wiki.ros.org/xacro">
+<robot name="kuka_kr150_2_robot" xmlns:xacro="http://wiki.ros.org/xacro">
   <xacro:include filename="$(find kr150_description)/urdf/kr150_2_macro.xacro" />
   <xacro:kuka_kr150_2 prefix=""/>

File: catkin_ws/src/KUKA_150/kr150_description/urdf/kr150_2_macro.xacro (robot description, xacro)
@@ -5,25 +5,35 @@
     <!-- base link -->
     <link name="${prefix}base_link">
-      <visual>
-        <origin rpy="0 0 0" xyz="0 0 0"/>
-        <geometry>
-          <mesh filename="package://kr150_description/meshes/kr150_2/visual/base_link.dae" />
-        </geometry>
-      </visual>
-      <collision>
-        <origin rpy="0 0 0" xyz="0 0 0"/>
-        <geometry>
-          <mesh filename="package://kr150_description/meshes/kr150_2/collision/base_link.stl" />
-        </geometry>
-      </collision>
       <inertial>
         <mass value="202.0"/>
         <!--          origen de esta inercia-->
         <origin rpy="0 0 0" xyz="0 0 0"/>
-        <inertia ixx="18.02664" ixy="-0.0638" ixz="-0.012" iyy="15.5177" iyz="-0.6815" izz="0.000202949"/>
-      </inertial>
+        <inertia ixx="18.02664"
+        ixy="-0.0638"
+        ixz="-0.012"
+        iyy="15.5177"
+        iyz="-0.6815"
+        izz="0.000202949"/>
+      </inertial>
+      <visual>
+        <origin rpy="0 0 0" xyz="0 0 0"/>
+        <geometry>
+          <mesh filename="package://kr150_description/meshes/kr150_2/visual/base_link.dae" />
+        </geometry>
+      </visual>
+      <collision>
+        <origin rpy="0 0 0" xyz="0 0 0"/>
+        <geometry>
+          <mesh filename="package://kr150_description/meshes/kr150_2/collision/base_link.stl" />
+        </geometry>
+      </collision>
     </link>
     <!-- link 1 (A1) -->
     <link name="${prefix}link_1">
+      <inertial>
+        <mass value="113.789"/>
+        <origin rpy="0 0 0" xyz="0 0 0"/>
+        <inertia ixx="44.25643" ixy="1.51540" ixz="-3.75190" iyy="38.43364" iyz="3.94701" izz="13.87916"/>
+      </inertial>
       <visual>
         <origin xyz="0 0 0" rpy="0 0 0"/>
@@ -38,12 +48,12 @@
         </geometry>
       </collision>
-      <inertial>
-        <mass value="113.789"/>
-        <origin rpy="0 0 0" xyz="0 0 0"/>
-        <inertia ixx="44.25643" ixy="1.51540" ixz="-3.75190" iyy="38.43364" iyz="3.94701" izz="13.87916"/>
-      </inertial>
     </link>
     <!-- link 2 -->
     <link name="${prefix}link_2">
+      <inertial>
+        <mass value="128.289"/>
+        <origin rpy="0 0 0" xyz="0 0 0"/>
+        <inertia ixx="222.75924" ixy="10.91733" ixz="37.96529" iyy="212.77949" iyz="55.85861" izz="26.73053"/>
+      </inertial>
       <visual>
         <origin xyz="0 0 0" rpy="0 0 0"/>
@@ -58,12 +68,12 @@
         </geometry>
       </collision>
-      <inertial>
-        <mass value="128.289"/>
-        <origin rpy="0 0 0" xyz="0 0 0"/>
-        <inertia ixx="222.75924" ixy="10.91733" ixz="37.96529" iyy="212.77949" iyz="55.85861" izz="26.73053"/>
-      </inertial>
     </link>
     <!-- link 3 -->
     <link name="${prefix}link_3">
+      <inertial>
+        <mass value="55.264" />
+        <origin rpy="0 0 0" xyz="0 0 0"/>
+        <inertia ixx="227.28356" ixy="-0.44413" ixz="2.39808" iyy="212.96072" iyz="50.90569" izz="14.91148"/>
+      </inertial>
       <visual>
         <origin xyz="0 0 0" rpy="0 0 0"/>
@@ -78,12 +88,12 @@
         </geometry>
       </collision>
-      <inertial>
-        <mass value="55.264" />
-        <origin rpy="0 0 0" xyz="0 0 0"/>
-        <inertia ixx="227.28356" ixy="-0.44413" ixz="2.39808" iyy="212.96072" iyz="50.90569" izz="14.91148"/>
-      </inertial>
     </link>
     <!-- link 4 -->
     <link name="${prefix}link_4">
+      <inertial>
+        <mass value="222.414"/>
+        <origin rpy="0 0 0" xyz="0 0 0"/>
+        <inertia ixx="116.69031" ixy=" -0.21747" ixz="0.31918" iyy="85.03211" iyz="51.42035" izz="32.00070"/>
+      </inertial>
       <visual>
         <origin xyz="0 0 0" rpy="0 0 0"/>
@@ -98,12 +108,12 @@
         </geometry>
       </collision>
-      <inertial>
-        <mass value="222.414"/>
-        <origin rpy="0 0 0" xyz="0 0 0"/>
-        <inertia ixx="116.69031" ixy=" -0.21747" ixz="0.31918" iyy="85.03211" iyz="51.42035" izz="32.00070"/>
-      </inertial>
     </link>
     <!-- link 5 -->
     <link name="${prefix}link_5">
+      <inertial>
+        <mass value="9.312"/>
+        <origin rpy="0 0 0" xyz="0 0 0"/>
+        <inertia ixx="56.09577" ixy="0.35043" ixz="0.47062" iyy="35.2848" iyz="27.05548" izz="20.8721"/>
+      </inertial>
       <visual>
         <origin xyz="0 0 0" rpy="0 0 0"/>
@@ -118,12 +128,12 @@
         </geometry>
       </collision>
-      <inertial>
-        <mass value="9.312"/>
-        <origin rpy="0 0 0" xyz="0 0 0"/>
-        <inertia ixx="56.09577" ixy="0.35043" ixz="0.47062" iyy="35.2848" iyz="27.05548" izz="20.8721"/>
-      </inertial>
     </link>
     <!-- link 6 -->
     <link name="${prefix}link_6">
+      <inertial>
+        <mass value="20.815"/>
+        <origin rpy="0 0 0" xyz="0 0 0"/>
+        <inertia ixx="5.33544" ixy="-0.000020453" ixz="0.000023961" iyy="3.08644" iyz="2.63404" izz="2.25310"/>
+      </inertial>
       <visual>
         <origin xyz="0 0 0" rpy="0 0 0"/>
@@ -138,9 +148,4 @@
         </geometry>
       </collision>
-      <inertial>
-        <mass value="20.815"/>
-        <origin rpy="0 0 0" xyz="0 0 0"/>
-        <inertia ixx="5.33544" ixy="-0.000020453" ixz="0.000023961" iyy="3.08644" iyz="2.63404" izz="2.25310"/>
-      </inertial>
     </link>
     <!-- tool link -->
@@ -155,5 +160,5 @@
       <child link="${prefix}link_1"/>
       <axis xyz="0 0 -1"/>
-      <limit effort="692" lower="${radians(-185)}" upper="${radians(185)}" velocity="${radians(110)}"/>
+      <limit effort="0" lower="${radians(-185)}" upper="${radians(185)}" velocity="${radians(110)}"/>
       <dynamics damping="0.0" friction="0.0"/>
     </joint>
@@ -164,5 +169,5 @@
       <child link="${prefix}link_2"/>
       <axis xyz="0 1 0"/>
-      <limit effort="574" lower="${radians(-146)}" upper="${radians(0)}" velocity="${radians(110)}"/>
+      <limit effort="0" lower="${radians(-146)}" upper="${radians(0)}" velocity="${radians(110)}"/>
       <dynamics damping="0.0" friction="0.0"/>
     </joint>
@@ -173,5 +178,5 @@
       <child link="${prefix}link_3"/>
       <axis xyz="0 1 0"/>
-      <limit effort="242" lower="${radians(-119)}" upper="${radians(155)}" velocity="${radians(100)}"/>
+      <limit effort="0" lower="${radians(-119)}" upper="${radians(155)}" velocity="${radians(100)}"/>
       <dynamics damping="0.0" friction="0.0"/>
     </joint>
@@ -182,5 +187,5 @@
       <child link="${prefix}link_4"/>
       <axis xyz="-1 0 0"/>
-      <limit effort="58" lower="${radians(-350)}" upper="${radians(350)}" velocity="${radians(170)}"/>
+      <limit effort="0" lower="${radians(-350)}" upper="${radians(350)}" velocity="${radians(170)}"/>
       <dynamics damping="0.0" friction="0.0"/>
     </joint>
@@ -191,5 +196,5 @@
       <child link="${prefix}link_5"/>
       <axis xyz="0 1 0"/>
-      <limit effort="29" lower="${radians(-125)}" upper="${radians(125)}" velocity="${radians(170)}"/>
+      <limit effort="0" lower="${radians(-125)}" upper="${radians(125)}" velocity="${radians(170)}"/>
       <dynamics damping="0.0" friction="0.0"/>
     </joint>
@@ -200,5 +205,5 @@
       <child link="${prefix}link_6"/>
       <axis xyz="-1 0 0"/>
-      <limit effort="29" lower="${radians(-350)}" upper="${radians(350)}" velocity="${radians(238)}"/>
+      <limit effort="0" lower="${radians(-350)}" upper="${radians(350)}" velocity="${radians(238)}"/>
       <dynamics damping="0.0" friction="0.0"/>
     </joint>

File: catkin_ws/src/KUKA_150/kr150_gazebo/urdf/gazebo.xacro (robot description, xacro)
@@ -3,5 +3,5 @@
   <!-- KR10 -->
   <xacro:include filename="$(find kr150_gazebo)/urdf/gazebo_transmission.xacro"/>
-  <xacro:kuka_kr150_robot prefix=""/>
+  <xacro:kuka_kr150_2_robot prefix=""/>
   <!-- Fix robot to Gazebo world -->
   <link name="world"/>

File: catkin_ws/src/KUKA_150/kr150_gazebo/urdf/gazebo_transmission.xacro (robot description, xacro)
@@ -2,5 +2,5 @@
 <robot xmlns:xacro="http://wiki.ros.org/xacro">
 <xacro:include filename="$(find kr150_description)/urdf/kr150_2_macro.xacro"/>
-<xacro:macro name="kuka_kr150_robot" params="prefix">
+<xacro:macro name="kuka_kr150_2_robot" params="prefix">
   <!-- get URDF description of KUKA KR150 model -->
   <xacro:kuka_kr150_2 prefix="${prefix}" />
