Commit message: Include Inertia and mass of links

File: catkin_ws/src/KUKA_150/kr150_description/urdf/kr150_2_macro.xacro (robot description, xacro)
@@ -17,9 +17,9 @@
         </geometry>
       </collision>
-      <!--inertial>
-        <mass value="23.085357"/>
-        <origin rpy="0 0 0" xyz="0 0 0"/>
-        <inertia ixx="0.343576" ixy="-0.000062" ixz="-0.002079" iyy="0.336217" iyz="-0.000014" izz="0.334050"/>
-      </inertial-->
+      <inertial>
+        <mass value="202"/>
+        <origin rpy="0 0 0" xyz="0 0 0"/>
+        <inertia ixx="18026640.942" ixy="-63776.874" ixz="-12034.191" iyy="15517698.140" iyz="-681592.618" izz="202.949"/>
+      </inertial>
     </link>
     <!-- link 1 (A1) -->
@@ -37,9 +37,9 @@
         </geometry>
       </collision>
-      <!--inertial>
-        <mass value="23.085357"/>
-        <origin rpy="0 0 0" xyz="0 0 0"/>
-        <inertia ixx="0.343576" ixy="-0.000062" ixz="-0.002079" iyy="0.336217" iyz="-0.000014" izz="0.334050"/>
-      </inertial-->
+      <inertial>
+        <mass value="113.789"/>
+        <origin rpy="0 0 0" xyz="0 0 0"/>
+        <inertia ixx="44256438.988" ixy="1515407.021" ixz="-3751903.667" iyy="38433645.587" iyz="3947019.941" izz="13879163.755"/>
+      </inertial>
     </link>
     <!-- link 2 -->
@@ -57,9 +57,9 @@
         </geometry>
       </collision>
-      <!--inertial>
-        <mass value="23.085357"/>
-        <origin rpy="0 0 0" xyz="0 0 0"/>
-        <inertia ixx="0.343576" ixy="-0.000062" ixz="-0.002079" iyy="0.336217" iyz="-0.000014" izz="0.334050"/>
-      </inertial-->
+      <inertial>
+        <mass value="128.289"/>
+        <origin rpy="0 0 0" xyz="0 0 0"/>
+        <inertia ixx="222759248.246" ixy="10917339.332" ixz="37965297.844 " iyy="212779494.067 " iyz="55858617.185" izz="26730538.796"/>
+      </inertial>
     </link>
     <!-- link 3 -->
@@ -77,9 +77,9 @@
         </geometry>
       </collision>
-      <!--inertial>
-        <mass value="23.085357"/>
-        <origin rpy="0 0 0" xyz="0 0 0"/>
-        <inertia ixx="0.343576" ixy="-0.000062" ixz="-0.002079" iyy="0.336217" iyz="-0.000014" izz="0.334050"/>
-      </inertial-->
+      <inertial>
+        <mass value="55.264" />
+        <origin rpy="0 0 0" xyz="0 0 0"/>
+        <inertia ixx="227283567.242 " ixy="-444134.292" ixz="2398080.124" iyy="212960722.458" iyz="50905692.306" izz="14911487.072"/>
+      </inertial>
     </link>
     <!-- link 4 -->
@@ -97,9 +97,9 @@
         </geometry>
       </collision>
-      <!--inertial>
-        <mass value="23.085357"/>
-        <origin rpy="0 0 0" xyz="0 0 0"/>
-        <inertia ixx="0.343576" ixy="-0.000062" ixz="-0.002079" iyy="0.336217" iyz="-0.000014" izz="0.334050"/>
-      </inertial-->
+      <inertial>
+        <mass value="222.414"/>
+        <origin rpy="0 0 0" xyz="0 0 0"/>
+        <inertia ixx="116690317.289 " ixy=" -217478.502" ixz="319180.825 " iyy="85032110.170" iyz="51420359.377" izz="32000704.547"/>
+      </inertial>
     </link>
     <!-- link 5 -->
@@ -117,9 +117,9 @@
         </geometry>
       </collision>
-      <!--inertial>
-        <mass value="23.085357"/>
-        <origin rpy="0 0 0" xyz="0 0 0"/>
-        <inertia ixx="0.343576" ixy="-0.000062" ixz="-0.002079" iyy="0.336217" iyz="-0.000014" izz="0.334050"/>
-      </inertial-->
+      <inertial>
+        <mass value="9.312"/>
+        <origin rpy="0 0 0" xyz="0 0 0"/>
+        <inertia ixx="56095774.637" ixy="350435.185" ixz="470622.777" iyy="35284894.395" iyz="27055480.349" izz="20872134.322"/>
+      </inertial>
     </link>
     <!-- link 6 -->
@@ -137,9 +137,9 @@
         </geometry>
       </collision>
-      <!--inertial>
+      <inertial>
         <mass value="23.085357"/>
         <origin rpy="0 0 0" xyz="0 0 0"/>
         <inertia ixx="0.343576" ixy="-0.000062" ixz="-0.002079" iyy="0.336217" iyz="-0.000014" izz="0.334050"/>
-      </inertial-->
+      </inertial>
     </link>
     <!-- tool link -->

Commit message: Advance until gazebo launch file. Did not run. MASS NOT UPDATED

File: catkin_ws/src/KUKA_150/kr150_description/urdf/kr150_2_macro.xacro (robot description, xacro)
@@ -19,6 +19,7 @@
       <inertial>
         <mass value="202"/>
-        <origin rpy="0 0 0" xyz="0 0 0"/>
-        <inertia ixx="18026640.942" ixy="-63776.874" ixz="-12034.191" iyy="15517698.140" iyz="-681592.618" izz="202.949"/>
+        <!--          origen de esta inercia-->
+        <origin rpy="0 0 0" xyz="0 0 0"/>
+        <inertia ixx="18.02664" ixy="-0.0638'" ixz="--0.012" iyy="15.5177" iyz="-0.6815" izz="0.000202949"/>
       </inertial>
     </link>
@@ -40,5 +41,5 @@
         <mass value="113.789"/>
         <origin rpy="0 0 0" xyz="0 0 0"/>
-        <inertia ixx="44256438.988" ixy="1515407.021" ixz="-3751903.667" iyy="38433645.587" iyz="3947019.941" izz="13879163.755"/>
+        <inertia ixx="44.25643" ixy="1.51540" ixz="-3.75190" iyy="38.43364" iyz="3.94701" izz="13.87916"/>
       </inertial>
     </link>
@@ -60,5 +61,5 @@
         <mass value="128.289"/>
         <origin rpy="0 0 0" xyz="0 0 0"/>
-        <inertia ixx="222759248.246" ixy="10917339.332" ixz="37965297.844 " iyy="212779494.067 " iyz="55858617.185" izz="26730538.796"/>
+        <inertia ixx="222.75924" ixy="10.91733" ixz="37.96529 " iyy="212.77949" iyz="55.85861" izz="26.73053"/>
       </inertial>
     </link>
@@ -80,5 +81,5 @@
         <mass value="55.264" />
         <origin rpy="0 0 0" xyz="0 0 0"/>
-        <inertia ixx="227283567.242 " ixy="-444134.292" ixz="2398080.124" iyy="212960722.458" iyz="50905692.306" izz="14911487.072"/>
+        <inertia ixx="227.28356" ixy="-0.44413" ixz="2.39808" iyy="212.96072" iyz="50.90569" izz="14.91148"/>
       </inertial>
     </link>
@@ -100,5 +101,5 @@
         <mass value="222.414"/>
         <origin rpy="0 0 0" xyz="0 0 0"/>
-        <inertia ixx="116690317.289 " ixy=" -217478.502" ixz="319180.825 " iyy="85032110.170" iyz="51420359.377" izz="32000704.547"/>
+        <inertia ixx="116.69031 " ixy=" -0.21747" ixz="0.31918" iyy="85.03211" iyz="51.42035" izz="32.00070"/>
       </inertial>
     </link>
@@ -120,5 +121,5 @@
         <mass value="9.312"/>
         <origin rpy="0 0 0" xyz="0 0 0"/>
-        <inertia ixx="56095774.637" ixy="350435.185" ixz="470622.777" iyy="35284894.395" iyz="27055480.349" izz="20872134.322"/>
+        <inertia ixx="56.09577" ixy="0.35043" ixz="0.47062" iyy="35.2848" iyz="27.05548" izz="20.8721"/>
       </inertial>
     </link>
@@ -155,4 +156,5 @@
       <axis xyz="0 0 -1"/>
       <limit effort="0" lower="${radians(-185)}" upper="${radians(185)}" velocity="${radians(110)}"/>
+      <dynamics damping="0.0" friction="0.0"/>
     </joint>
     <!-- joint 2 (A2) -->
@@ -163,4 +165,5 @@
       <axis xyz="0 1 0"/>
       <limit effort="0" lower="${radians(-146)}" upper="${radians(0)}" velocity="${radians(110)}"/>
+      <dynamics damping="0.0" friction="0.0"/>
     </joint>
     <!-- joint 3 (A3) -->
@@ -171,4 +174,5 @@
       <axis xyz="0 1 0"/>
       <limit effort="0" lower="${radians(-119)}" upper="${radians(155)}" velocity="${radians(100)}"/>
+      <dynamics damping="0.0" friction="0.0"/>
     </joint>
     <!-- joint 4 (A4) -->
@@ -179,4 +183,5 @@
       <axis xyz="-1 0 0"/>
       <limit effort="0" lower="${radians(-350)}" upper="${radians(350)}" velocity="${radians(170)}"/>
+      <dynamics damping="0.0" friction="0.0"/>
     </joint>
     <!-- joint 5 (A5) -->
@@ -187,4 +192,5 @@
       <axis xyz="0 1 0"/>
       <limit effort="0" lower="${radians(-125)}" upper="${radians(125)}" velocity="${radians(170)}"/>
+      <dynamics damping="0.0" friction="0.0"/>
     </joint>
     <!-- joint 6 (A6) -->
@@ -195,4 +201,5 @@
       <axis xyz="-1 0 0"/>
       <limit effort="0" lower="${radians(-350)}" upper="${radians(350)}" velocity="${radians(238)}"/>
+      <dynamics damping="0.0" friction="0.0"/>
     </joint>
     <!-- tool frame - fixed frame -->

Commit message: Tiny test changes. Still not running. Pt2

File: catkin_ws/src/KUKA_150/kr150_description/urdf/kr150_2_macro.xacro (robot description, xacro)
@@ -21,5 +21,5 @@
         <!--          origen de esta inercia-->
         <origin rpy="0 0 0" xyz="0 0 0"/>
-        <inertia ixx="18.02664" ixy="-0.0638'" ixz="--0.012" iyy="15.5177" iyz="-0.6815" izz="0.000202949"/>
+        <inertia ixx="18.02664" ixy="-0.0638" ixz="-0.012" iyy="15.5177" iyz="-0.6815" izz="0.000202949"/>
       </inertial>
     </link>
@@ -61,5 +61,5 @@
         <mass value="128.289"/>
         <origin rpy="0 0 0" xyz="0 0 0"/>
-        <inertia ixx="222.75924" ixy="10.91733" ixz="37.96529 " iyy="212.77949" iyz="55.85861" izz="26.73053"/>
+        <inertia ixx="222.75924" ixy="10.91733" ixz="37.96529" iyy="212.77949" iyz="55.85861" izz="26.73053"/>
       </inertial>
     </link>
@@ -101,5 +101,5 @@
         <mass value="222.414"/>
         <origin rpy="0 0 0" xyz="0 0 0"/>
-        <inertia ixx="116.69031 " ixy=" -0.21747" ixz="0.31918" iyy="85.03211" iyz="51.42035" izz="32.00070"/>
+        <inertia ixx="116.69031" ixy=" -0.21747" ixz="0.31918" iyy="85.03211" iyz="51.42035" izz="32.00070"/>
       </inertial>
     </link>
@@ -139,7 +139,7 @@
       </collision>
       <inertial>
-        <mass value="23.085357"/>
-        <origin rpy="0 0 0" xyz="0 0 0"/>
-        <inertia ixx="0.343576" ixy="-0.000062" ixz="-0.002079" iyy="0.336217" iyz="-0.000014" izz="0.334050"/>
+        <mass value="20.815"/>
+        <origin rpy="0 0 0" xyz="0 0 0"/>
+        <inertia ixx="5.33544" ixy="-0.000020453" ixz="0.000023961" iyy="3.08644" iyz="2.63404" izz="2.25310"/>
       </inertial>
     </link>

Commit message: Not running pt3

File: catkin_ws/src/KUKA_150/kr150_description/urdf/kr150_2_macro.xacro (robot description, xacro)
@@ -155,5 +155,5 @@
       <child link="${prefix}link_1"/>
       <axis xyz="0 0 -1"/>
-      <limit effort="0" lower="${radians(-185)}" upper="${radians(185)}" velocity="${radians(110)}"/>
+      <limit effort="692" lower="${radians(-185)}" upper="${radians(185)}" velocity="${radians(110)}"/>
       <dynamics damping="0.0" friction="0.0"/>
     </joint>
@@ -164,5 +164,5 @@
       <child link="${prefix}link_2"/>
       <axis xyz="0 1 0"/>
-      <limit effort="0" lower="${radians(-146)}" upper="${radians(0)}" velocity="${radians(110)}"/>
+      <limit effort="574" lower="${radians(-146)}" upper="${radians(0)}" velocity="${radians(110)}"/>
       <dynamics damping="0.0" friction="0.0"/>
     </joint>
@@ -173,5 +173,5 @@
       <child link="${prefix}link_3"/>
       <axis xyz="0 1 0"/>
-      <limit effort="0" lower="${radians(-119)}" upper="${radians(155)}" velocity="${radians(100)}"/>
+      <limit effort="242" lower="${radians(-119)}" upper="${radians(155)}" velocity="${radians(100)}"/>
       <dynamics damping="0.0" friction="0.0"/>
     </joint>
@@ -182,5 +182,5 @@
       <child link="${prefix}link_4"/>
       <axis xyz="-1 0 0"/>
-      <limit effort="0" lower="${radians(-350)}" upper="${radians(350)}" velocity="${radians(170)}"/>
+      <limit effort="58" lower="${radians(-350)}" upper="${radians(350)}" velocity="${radians(170)}"/>
       <dynamics damping="0.0" friction="0.0"/>
     </joint>
@@ -191,5 +191,5 @@
       <child link="${prefix}link_5"/>
       <axis xyz="0 1 0"/>
-      <limit effort="0" lower="${radians(-125)}" upper="${radians(125)}" velocity="${radians(170)}"/>
+      <limit effort="29" lower="${radians(-125)}" upper="${radians(125)}" velocity="${radians(170)}"/>
       <dynamics damping="0.0" friction="0.0"/>
     </joint>
@@ -200,5 +200,5 @@
       <child link="${prefix}link_6"/>
       <axis xyz="-1 0 0"/>
-      <limit effort="0" lower="${radians(-350)}" upper="${radians(350)}" velocity="${radians(238)}"/>
+      <limit effort="29" lower="${radians(-350)}" upper="${radians(350)}" velocity="${radians(238)}"/>
       <dynamics damping="0.0" friction="0.0"/>
     </joint>

Commit message: Gazebo utils cloned, kuka experimental  cloned

File: catkin_ws/src/KUKA_150/kr150_description/urdf/kr150_2_macro.xacro (robot description, xacro)
@@ -18,5 +18,5 @@
       </collision>
       <inertial>
-        <mass value="202"/>
+        <mass value="202.0"/>
         <!--          origen de esta inercia-->
         <origin rpy="0 0 0" xyz="0 0 0"/>

Commit message: banda

File: catkin_ws/src/KUKA_150/kr150_description/urdf/kr150_2_macro.xacro (robot description, xacro)
@@ -17,9 +17,10 @@
         </geometry>
       </collision>
-      <!--inertial>
-        <mass value="23.085357"/>
-        <origin rpy="0 0 0" xyz="0 0 0"/>
-        <inertia ixx="0.343576" ixy="-0.000062" ixz="-0.002079" iyy="0.336217" iyz="-0.000014" izz="0.334050"/>
-      </inertial-->
+      <inertial>
+        <mass value="202"/>
+        <!--          origen de esta inercia-->
+        <origin rpy="0 0 0" xyz="0 0 0"/>
+        <inertia ixx="18.02664" ixy="-0.0638" ixz="-0.012" iyy="15.5177" iyz="-0.6815" izz="0.000202949"/>
+      </inertial>
     </link>
     <!-- link 1 (A1) -->
@@ -37,9 +38,9 @@
         </geometry>
       </collision>
-      <!--inertial>
-        <mass value="23.085357"/>
-        <origin rpy="0 0 0" xyz="0 0 0"/>
-        <inertia ixx="0.343576" ixy="-0.000062" ixz="-0.002079" iyy="0.336217" iyz="-0.000014" izz="0.334050"/>
-      </inertial-->
+      <inertial>
+        <mass value="113.789"/>
+        <origin rpy="0 0 0" xyz="0 0 0"/>
+        <inertia ixx="44.25643" ixy="1.51540" ixz="-3.75190" iyy="38.43364" iyz="3.94701" izz="13.87916"/>
+      </inertial>
     </link>
     <!-- link 2 -->
@@ -57,9 +58,9 @@
         </geometry>
       </collision>
-      <!--inertial>
-        <mass value="23.085357"/>
-        <origin rpy="0 0 0" xyz="0 0 0"/>
-        <inertia ixx="0.343576" ixy="-0.000062" ixz="-0.002079" iyy="0.336217" iyz="-0.000014" izz="0.334050"/>
-      </inertial-->
+      <inertial>
+        <mass value="128.289"/>
+        <origin rpy="0 0 0" xyz="0 0 0"/>
+        <inertia ixx="222.75924" ixy="10.91733" ixz="37.96529" iyy="212.77949" iyz="55.85861" izz="26.73053"/>
+      </inertial>
     </link>
     <!-- link 3 -->
@@ -77,9 +78,9 @@
         </geometry>
       </collision>
-      <!--inertial>
-        <mass value="23.085357"/>
-        <origin rpy="0 0 0" xyz="0 0 0"/>
-        <inertia ixx="0.343576" ixy="-0.000062" ixz="-0.002079" iyy="0.336217" iyz="-0.000014" izz="0.334050"/>
-      </inertial-->
+      <inertial>
+        <mass value="55.264" />
+        <origin rpy="0 0 0" xyz="0 0 0"/>
+        <inertia ixx="227.28356" ixy="-0.44413" ixz="2.39808" iyy="212.96072" iyz="50.90569" izz="14.91148"/>
+      </inertial>
     </link>
     <!-- link 4 -->
@@ -97,9 +98,9 @@
         </geometry>
       </collision>
-      <!--inertial>
-        <mass value="23.085357"/>
-        <origin rpy="0 0 0" xyz="0 0 0"/>
-        <inertia ixx="0.343576" ixy="-0.000062" ixz="-0.002079" iyy="0.336217" iyz="-0.000014" izz="0.334050"/>
-      </inertial-->
+      <inertial>
+        <mass value="222.414"/>
+        <origin rpy="0 0 0" xyz="0 0 0"/>
+        <inertia ixx="116.69031" ixy=" -0.21747" ixz="0.31918" iyy="85.03211" iyz="51.42035" izz="32.00070"/>
+      </inertial>
     </link>
     <!-- link 5 -->
@@ -117,9 +118,9 @@
         </geometry>
       </collision>
-      <!--inertial>
-        <mass value="23.085357"/>
-        <origin rpy="0 0 0" xyz="0 0 0"/>
-        <inertia ixx="0.343576" ixy="-0.000062" ixz="-0.002079" iyy="0.336217" iyz="-0.000014" izz="0.334050"/>
-      </inertial-->
+      <inertial>
+        <mass value="9.312"/>
+        <origin rpy="0 0 0" xyz="0 0 0"/>
+        <inertia ixx="56.09577" ixy="0.35043" ixz="0.47062" iyy="35.2848" iyz="27.05548" izz="20.8721"/>
+      </inertial>
     </link>
     <!-- link 6 -->
@@ -137,9 +138,9 @@
         </geometry>
       </collision>
-      <!--inertial>
-        <mass value="23.085357"/>
-        <origin rpy="0 0 0" xyz="0 0 0"/>
-        <inertia ixx="0.343576" ixy="-0.000062" ixz="-0.002079" iyy="0.336217" iyz="-0.000014" izz="0.334050"/>
-      </inertial-->
+      <inertial>
+        <mass value="20.815"/>
+        <origin rpy="0 0 0" xyz="0 0 0"/>
+        <inertia ixx="5.33544" ixy="-0.000020453" ixz="0.000023961" iyy="3.08644" iyz="2.63404" izz="2.25310"/>
+      </inertial>
     </link>
     <!-- tool link -->
@@ -154,5 +155,6 @@
       <child link="${prefix}link_1"/>
       <axis xyz="0 0 -1"/>
-      <limit effort="0" lower="${radians(-185)}" upper="${radians(185)}" velocity="${radians(110)}"/>
+      <limit effort="692" lower="${radians(-185)}" upper="${radians(185)}" velocity="${radians(110)}"/>
+      <dynamics damping="0.0" friction="0.0"/>
     </joint>
     <!-- joint 2 (A2) -->
@@ -162,5 +164,6 @@
       <child link="${prefix}link_2"/>
       <axis xyz="0 1 0"/>
-      <limit effort="0" lower="${radians(-146)}" upper="${radians(0)}" velocity="${radians(110)}"/>
+      <limit effort="574" lower="${radians(-146)}" upper="${radians(0)}" velocity="${radians(110)}"/>
+      <dynamics damping="0.0" friction="0.0"/>
     </joint>
     <!-- joint 3 (A3) -->
@@ -170,5 +173,6 @@
       <child link="${prefix}link_3"/>
       <axis xyz="0 1 0"/>
-      <limit effort="0" lower="${radians(-119)}" upper="${radians(155)}" velocity="${radians(100)}"/>
+      <limit effort="242" lower="${radians(-119)}" upper="${radians(155)}" velocity="${radians(100)}"/>
+      <dynamics damping="0.0" friction="0.0"/>
     </joint>
     <!-- joint 4 (A4) -->
@@ -178,5 +182,6 @@
       <child link="${prefix}link_4"/>
       <axis xyz="-1 0 0"/>
-      <limit effort="0" lower="${radians(-350)}" upper="${radians(350)}" velocity="${radians(170)}"/>
+      <limit effort="58" lower="${radians(-350)}" upper="${radians(350)}" velocity="${radians(170)}"/>
+      <dynamics damping="0.0" friction="0.0"/>
     </joint>
     <!-- joint 5 (A5) -->
@@ -186,5 +191,6 @@
       <child link="${prefix}link_5"/>
       <axis xyz="0 1 0"/>
-      <limit effort="0" lower="${radians(-125)}" upper="${radians(125)}" velocity="${radians(170)}"/>
+      <limit effort="29" lower="${radians(-125)}" upper="${radians(125)}" velocity="${radians(170)}"/>
+      <dynamics damping="0.0" friction="0.0"/>
     </joint>
     <!-- joint 6 (A6) -->
@@ -194,5 +200,6 @@
       <child link="${prefix}link_6"/>
       <axis xyz="-1 0 0"/>
-      <limit effort="0" lower="${radians(-350)}" upper="${radians(350)}" velocity="${radians(238)}"/>
+      <limit effort="29" lower="${radians(-350)}" upper="${radians(350)}" velocity="${radians(238)}"/>
+      <dynamics damping="0.0" friction="0.0"/>
     </joint>
     <!-- tool frame - fixed frame -->

Commit message: Gazebo running, main running with arguments (camera, gripper)

File: catkin_ws/src/KUKA_150/kr150_description/urdf/kr150_2_macro.xacro (robot description, xacro)
@@ -160,5 +160,8 @@
       <child link="${prefix}link_1"/>
       <axis xyz="0 0 -1"/>
-      <limit effort="0" lower="${radians(-185)}" upper="${radians(185)}" velocity="${radians(110)}"/>
+      <limit effort="0"
+      lower="${radians(-185)}"
+      upper="${radians(185)}"
+      velocity="${radians(110)}"/>
       <dynamics damping="0.0" friction="0.0"/>
     </joint>
@@ -169,5 +172,6 @@
       <child link="${prefix}link_2"/>
       <axis xyz="0 1 0"/>
-      <limit effort="0" lower="${radians(-146)}" upper="${radians(0)}" velocity="${radians(110)}"/>
+      <limit effort="0"
+      lower="${radians(-146)}" upper="${radians(0)}" velocity="${radians(110)}"/>
       <dynamics damping="0.0" friction="0.0"/>
     </joint>
