Commit message: Conveyor belt included, arguments functional. Controllable speed, spawnable boxes.

File: catkin_ws/src/KUKA_150/kr150_gazebo/urdf/camera.xacro (robot description, xacro)
@@ -14,5 +14,5 @@
         <box size="0.1 0.7 0.7"/>
       </geometry>
-      <material name="grey"/>
+      <material name="gray"/>
     </visual>
     <inertial>
@@ -31,5 +31,5 @@
   <joint name="camera_joint" type="fixed">
     <axis xyz="0 0 0"/>
-    <origin rpy="0 1.5708 0" xyz="0.5 0 2.0"/>
+    <origin rpy="0 1.5708 0" xyz="0.5 0 3.5"/>
     <parent link="base_link"/>
     <child link="camera"/>

File: catkin_ws/src/KUKA_150/kr150_gazebo/urdf/kr150_main.xacro (robot description, xacro)
@@ -4,4 +4,5 @@
   <xacro:arg name="gripper_2f" default="false"/>
   <xacro:include filename="$(find kr150_gazebo)/urdf/gazebo.xacro"/>
+  <xacro:include filename="$(find kr150_gazebo)/urdf/banda.xacro"/>
   <!-- camera -->
   <xacro:if value="$(arg camera)">

Commit message: Moveit, base poses, incorporated colored camera with no algorithm

File: catkin_ws/src/KUKA_150/kr150_gazebo/urdf/camera.xacro (robot description, xacro)
@@ -31,5 +31,5 @@
   <joint name="camera_joint" type="fixed">
     <axis xyz="0 0 0"/>
-    <origin rpy="0 1.5708 0" xyz="0.5 0 3.5"/>
+    <origin rpy="0 1.5708 0" xyz="0 -2 3.5"/>
     <parent link="base_link"/>
     <child link="camera"/>

File: catkin_ws/src/KUKA_150/kr150_gazebo/urdf/kr150_main.urdf (robot description, URDF)
Before this commit: robot kr150_main, 25 links, 24 joints
Links:
- added link belt_moving, mass 100; collision box size=0.425 2.4 0.001; visual box size=0.425 2.4 0.001
- added link belt_visual, mass 71.953; collision mesh filename=package://kr150_description/meshes/conveyor/conveyor_belt.s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 scale=1 2 1; visual mesh filename=package://kr150_description/meshes/conveyor/conveyor_belt.s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 scale=1 2 1
Joints:
- added joint banda_fixed: type fixed, parent world, child belt_visual, origin xyz=0.0 -2.0 0.0 rpy=0.0 0.0 1.57
- added joint belt_joint: type prismatic, parent belt_visual, child belt_moving, origin xyz=0.0 0.0 0.74 rpy=0.0 0.0 0.0, axis 0 1 0, limit lower=0.0 upper=1 effort=1000 velocity=1000
- joint camera_joint: origin xyz=0.5 0 2.0 rpy=0 1.5708 0 -> xyz=0 -2 3.5 rpy=0 1.5708 0

File: catkin_ws/src/KUKA_150/kr150_gazebo/urdf/kr150_main.xacro (robot description, xacro)
@@ -1,8 +1,10 @@
 <?xml version="1.0" ?>
 <robot name="kr150_main" xmlns:xacro="http://ros.org/wiki/xacro">
-  <xacro:arg name="camera" default="false"/>
+  <xacro:arg name="camera" default="true"/>
   <xacro:arg name="gripper_2f" default="false"/>
+  <xacro:arg name="conveyor" default="false"/>
+  <xacro:arg name="conveyor_RED" default="false"/>
   <xacro:include filename="$(find kr150_gazebo)/urdf/gazebo.xacro"/>
-  <xacro:include filename="$(find kr150_gazebo)/urdf/banda.xacro"/>
+  <!--<xacro:include filename="$(find kr150_gazebo)/urdf/banda.xacro"/>-->
   <!-- camera -->
   <xacro:if value="$(arg camera)">
@@ -13,3 +15,11 @@
     <xacro:include filename="$(find kr150_gazebo)/urdf/gazebo_2f.xacro"/>
   </xacro:if>
+  <!-- conveyor -->
+  <xacro:if value="$(arg conveyor)">
+    <xacro:include filename="$(find kr150_gazebo)/urdf/banda.xacro"/>
+  </xacro:if>
+  <!-- conveyor RED-->
+  <xacro:if value="$(arg conveyor_RED)">
+    <xacro:include filename="$(find kr150_gazebo)/urdf/banda_RED.xacro"/>
+  </xacro:if>
 </robot>
