Commit message: moveit poses

File: catkin_ws/src/KUKA_150/kr150_gazebo/urdf/banda.xacro (robot description, xacro)
@@ -55,5 +55,5 @@
 			<inertia ixx="0.0" ixy="0.0" ixz="0.0" iyy="0.0" iyz="0.0" izz="0.0"/>
 		</inertial>
-		<visual>
+		<!--<visual>
 			<origin xyz="0.0 0.0 0.0005" rpy="0.0 0.0 0.0"/>
 			<geometry>
@@ -63,5 +63,5 @@
 				<color rgba="1 0 1 1" />
 			</material>
-		</visual>
+		</visual>-->
 		<collision>
 			<origin xyz="0.0 0.0 0.0005" rpy="0.0 0.0 0.0"/>

File: catkin_ws/src/KUKA_150/kr150_gazebo/urdf/camera.xacro (robot description, xacro)
@@ -31,5 +31,5 @@
   <joint name="camera_joint" type="fixed">
     <axis xyz="0 0 0"/>
-    <origin rpy="0 1.5708 0" xyz="0 -2 3.5"/>
+    <origin rpy="0 1.5708 0" xyz="0 -2 2.5"/>
     <parent link="base_link"/>
     <child link="camera"/>

File: catkin_ws/src/KUKA_150/kr150_gazebo/urdf/gazebo_2f.urdf (robot description, URDF)
Before this commit: robot kuka_kr150_gripper, 23 links, 22 joints
Links:
- removed link base
- removed link base_link
- removed link flange
- removed link link_1
- removed link link_2
- removed link link_3
- removed link link_4
- removed link link_5
- removed link link_6
- removed link tool0
- removed link world
Joints:
- removed joint base_link-base
- removed joint flange-tool0
- removed joint joint_a1
- removed joint joint_a2
- removed joint joint_a3
- removed joint joint_a4
- removed joint joint_a5
- removed joint joint_a6
- removed joint joint_a6-flange
- removed joint world-base_link-fixed

File: catkin_ws/src/KUKA_150/kr150_gazebo/urdf/kr150_main.xacro (robot description, xacro)
@@ -4,5 +4,5 @@
   <xacro:arg name="gripper_2f" default="false"/>
   <xacro:arg name="conveyor" default="false"/>
-  <xacro:arg name="conveyor_RED" default="false"/>
+  <!--<xacro:arg name="conveyor_RED" default="false"/>-->
   <xacro:include filename="$(find kr150_gazebo)/urdf/gazebo.xacro"/>
   <!--<xacro:include filename="$(find kr150_gazebo)/urdf/banda.xacro"/>-->
@@ -19,7 +19,7 @@
     <xacro:include filename="$(find kr150_gazebo)/urdf/banda.xacro"/>
   </xacro:if>
-  <!-- conveyor RED-->
+  <!-- conveyor RED
   <xacro:if value="$(arg conveyor_RED)">
     <xacro:include filename="$(find kr150_gazebo)/urdf/banda_RED.xacro"/>
-  </xacro:if>
+  </xacro:if>-->
 </robot>
