Commit message: second try, failed attempt

File: catkin_ws/src/KUKA_150/kr150_gazebo/urdf/gazebo_2f.urdf (robot description, URDF)
Before this commit: robot kuka_kr150_gripper, 12 links, 12 joints
Links:
- link left_inner_finger_pad: mass None -> 0.1
- link right_inner_finger_pad: mass None -> 0.1

File: catkin_ws/src/KUKA_150/kr150_gazebo/urdf/gazebo_2f.xacro (robot description, xacro)
@@ -1,4 +1,4 @@
 <?xml version="1.0" ?>
-<robot name="kuka_kr150_gripper" xmlns:xacro="http://ros.org/wiki/xacro">
+<robot name="kuka_kr150_2_gripper" xmlns:xacro="http://ros.org/wiki/xacro">
   <!--<xacro:include filename="$(find kr150_gazebo)/urdf/gazebo.xacro"/>-->
   <xacro:include filename="$(find robotiq_2f_85_description)/urdf/robotiq_2F_85.xacro"/>

File: catkin_ws/src/KUKA_150/kr150_gazebo/urdf/transmission_2f.xacro (robot description, xacro)
@@ -89,5 +89,5 @@
     <plugin filename="libgazebo_grasp_fix.so" name="gazebo_grasp_fix">
       <arm>
-        <arm_name>kuka_kr150_2_robot</arm_name>
+        <arm_name>kuka_kr150_grasp</arm_name>
         <palm_link>link_6</palm_link>
         <gripper_link>left_outer_knuckle</gripper_link>
